File: Hardware/circuit board design v2.1/gps.kicad_sch (KiCad schematic)
At the start: 4 parts, among them U12 L80-R

Commit message: Renamed pins in stm32cubeide and finished routing for V2.1
Connections:
- net reset_gps renamed GPS_Reset
- net rx_gps renamed GPS_UART_RX_Module
- net tx_gps renamed GPS_UART_TX_Module
Changed lines of the file:
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@@
     (stroke (width 0) (type default) (color 0 0 0 0))
   )
-  (hierarchical_label "tx_gps" (shape output) (at 119.38 73.66 0)
+  (hierarchical_label "GPS_UART_TX_Module" (shape output) (at 119.38 73.66 0)
     (effects (font (size 1.27 1.27)) (justify left))
   )
-  (hierarchical_label "reset_gps" (shape input) (at 121.92 83.82 0)
+  (hierarchical_label "GPS_Reset" (shape input) (at 121.92 83.82 0)
     (effects (font (size 1.27 1.27)) (justify left))
   )
-  (hierarchical_label "rx_gps" (shape input) (at 119.38 76.2 0)
+  (hierarchical_label "GPS_UART_RX_Module" (shape input) (at 119.38 76.2 0)
     (effects (font (size 1.27 1.27)) (justify left))
   )

Commit message: PCB V2.1 sent for manufacture
Parts:
- U12: value L80-R -> L80-R GPS
Changed lines of the file:
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@@
       (effects (font (size 1.27 1.27)) (justify left))
     )
-    (property "Value" "L80-R" (id 1) (at 101.0794 93.98 0)
+    (property "Value" "L80-R GPS" (id 1) (at 101.0794 93.98 0)
       (effects (font (size 1.27 1.27)) (justify left))
     )
