File: Hardware/circuit board design v2.1/power_supply.kicad_sch (KiCad schematic)
At the start: 11 parts, among them J2 Conn_01x02, J3 105017-0001, U5 STF202-22T1G, U6 MAX40203_SOT23, U7 NCP161ASN330T1G

Commit message: Renamed pins in stm32cubeide and finished routing for V2.1
Connections:
- net PWR_BVOLTS renamed Battery_Voltage
- net usb_d+ renamed USB_D+
- net usb_d- renamed USB_D-
Changed lines of the file:
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@@
   (junction (at 59.69 53.34) (diameter 0) (color 0 0 0 0)
   )
-  (junction (at 186.69 48.26) (diameter 0) (color 0 0 0 0)
-  )
   (junction (at 227.33 100.33) (diameter 0) (color 0 0 0 0)
+  )
+  (junction (at 147.32 66.04) (diameter 0) (color 0 0 0 0)
   )
   (no_connect (at 59.69 48.26))
@@
     (stroke (width 0) (type default) (color 0 0 0 0))
   )
+  (wire (pts (xy 147.32 66.04) (xy 166.37 66.04))
+    (stroke (width 0) (type default) (color 0 0 0 0))
+  )
   (wire (pts (xy 227.33 100.33) (xy 227.33 101.6))
     (stroke (width 0) (type default) (color 0 0 0 0))
@@
     (stroke (width 0) (type default) (color 0 0 0 0))
   )
-  (wire (pts (xy 181.61 48.26) (xy 186.69 48.26))
-    (stroke (width 0) (type default) (color 0 0 0 0))
-  )
   (wire (pts (xy 184.15 100.33) (xy 187.96 100.33))
     (stroke (width 0) (type default) (color 0 0 0 0))
@@
     (stroke (width 0) (type default) (color 0 0 0 0))
   )
-  (wire (pts (xy 186.69 48.26) (xy 187.96 48.26))
+  (wire (pts (xy 181.61 48.26) (xy 187.96 48.26))
     (stroke (width 0) (type default) (color 0 0 0 0))
   )
@@
     (stroke (width 0) (type default) (color 0 0 0 0))
   )
-  (wire (pts (xy 125.73 66.04) (xy 166.37 66.04))
-    (stroke (width 0) (type default) (color 0 0 0 0))
-  )
-  (wire (pts (xy 125.73 53.34) (xy 144.78 53.34))
+  (wire (pts (xy 125.73 66.04) (xy 147.32 66.04))
+    (stroke (width 0) (type default) (color 0 0 0 0))
+  )
+  (wire (pts (xy 125.73 53.34) (xy 143.51 53.34))
     (stroke (width 0) (type default) (color 0 0 0 0))
   )
@@
     (effects (font (size 1.27 1.27)) (justify left bottom))
   )
-  (hierarchical_label "usb_d-" (shape bidirectional) (at 144.78 53.34 0)
+  (hierarchical_label "USB_D-" (shape bidirectional) (at 143.51 53.34 0)
     (effects (font (size 1.27 1.27)) (justify left))
   )
-  (hierarchical_label "PWR_BVOLTS" (shape output) (at 110.49 118.11 180)
+  (hierarchical_label "Battery_Voltage" (shape output) (at 110.49 118.11 180)
     (effects (font (size 1.27 1.27)) (justify right))
   )
-  (hierarchical_label "usb_d+" (shape bidirectional) (at 143.51 40.64 0)
+  (hierarchical_label "USB_D+" (shape bidirectional) (at 143.51 40.64 0)
     (effects (font (size 1.27 1.27)) (justify left))
   )
@@
     (pin "2")
   )
-  (symbol (lib_id "power:PWR_FLAG") (at 186.69 48.26 0) (unit 1)
-    (in_bom yes) (on_board yes) (fields_autoplaced)
-    (property "Reference" "#FLG0102" (id 0) (at 186.69 46.355 0)
-      (effects (font (size 1.27 1.27)) hide)
-    )
-    (property "Value" "PWR_FLAG" (id 1) (at 189.23 46.9899 0)
-      (effects (font (size 1.27 1.27)) (justify left))
-    )
-    (property "Footprint" "" (id 2) (at 186.69 48.26 0)
-      (effects (font (size 1.27 1.27)) hide)
-    )
-    (property "Datasheet" "~" (id 3) (at 186.69 48.26 0)
-      (effects (font (size 1.27 1.27)) hide)
-    )
+  (symbol (lib_id "power:PWR_FLAG") (at 147.32 66.04 0) (unit 1)
+    (in_bom yes) (on_board yes) (fields_autoplaced)
+    (property "Reference" "#FLG0102" (id 0) (at 147.32 64.135 0)
+      (effects (font (size 1.27 1.27)) hide)
+    )
+    (property "Value" "PWR_FLAG" (id 1) (at 149.86 64.7699 0)
+      (effects (font (size 1.27 1.27)) (justify left))
+    )
+    (property "Footprint" "" (id 2) (at 147.32 66.04 0)
+      (effects (font (size 1.27 1.27)) hide)
+    )
+    (property "Datasheet" "~" (id 3) (at 147.32 66.04 0)
+      (effects (font (size 1.27 1.27)) hide)
+    )

Commit message: Added interupt pins to from BMI088 and LIS
Other:
- moved on the sheet: C16, C3, C4, D1, J2, J3, R1, R2, U5, U6, U7

Commit message: PCB V2.1 sent for manufacture
Parts:
- C16: value 4.7uF -> 4.7uF Tantalum Capacitor
- D1: value DFLS130L -> DFLS130L Schottkey Diode
- J2: value Conn_01x02 -> JST_PH_S2B-PH-K_1x02_P2.00mm_Horizontal
- J3: value 105017-0001 -> 105017-0001 Micro USB Conn
- U5: value STF202-22T1G -> STF202-22T1G ESD/EMI Chip
- U6: value MAX40203_SOT23 -> MAX40203_SOT23 Ideal Diode
- U7: value NCP161ASN330T1G -> NCP161ASN330T1G LDO
Other:
- moved on the sheet: C16
Changed lines of the file:
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@@
   (junction (at 54.61 78.74) (diameter 0) (color 0 0 0 0)
   )
+  (junction (at 128.27 130.81) (diameter 0) (color 0 0 0 0)
+  )
+  (junction (at 179.07 113.03) (diameter 0) (color 0 0 0 0)
+  )
+  (junction (at 54.61 73.66) (diameter 0) (color 0 0 0 0)
+  )
+  (junction (at 54.61 81.28) (diameter 0) (color 0 0 0 0)
+  )
+  (junction (at 54.61 68.58) (diameter 0) (color 0 0 0 0)
+  )
+  (junction (at 187.96 113.03) (diameter 0) (color 0 0 0 0)
+  )
+  (junction (at 182.88 113.03) (diameter 0) (color 0 0 0 0)
+  )
   (junction (at 223.52 113.03) (diameter 0) (color 0 0 0 0)
   )
-  (junction (at 128.27 130.81) (diameter 0) (color 0 0 0 0)
-  )
-  (junction (at 179.07 113.03) (diameter 0) (color 0 0 0 0)
-  )
-  (junction (at 54.61 73.66) (diameter 0) (color 0 0 0 0)
-  )
-  (junction (at 54.61 81.28) (diameter 0) (color 0 0 0 0)
-  )
-  (junction (at 54.61 68.58) (diameter 0) (color 0 0 0 0)
-  )
-  (junction (at 187.96 113.03) (diameter 0) (color 0 0 0 0)
-  )
-  (junction (at 182.88 113.03) (diameter 0) (color 0 0 0 0)
-  )
   (junction (at 128.27 113.03) (diameter 0) (color 0 0 0 0)
   )
@@
   )
   (no_connect (at 54.61 60.96))
-  (wire (pts (xy 234.95 118.11) (xy 234.95 119.38))
-    (stroke (width 0) (type default) (color 0 0 0 0))
-  )
   (wire (pts (xy 161.29 60.96) (xy 161.29 78.74))
     (stroke (width 0) (type default) (color 0 0 0 0))
@@
     (stroke (width 0) (type default) (color 0 0 0 0))
   )
-  (wire (pts (xy 223.52 113.03) (xy 234.95 113.03))
-    (stroke (width 0) (type default) (color 0 0 0 0))
-  )
   (wire (pts (xy 128.27 113.03) (xy 147.32 113.03))
     (stroke (width 0) (type default) (color 0 0 0 0))
@@
     (stroke (width 0) (type default) (color 0 0 0 0))
   )
+  (wire (pts (xy 234.95 114.3) (xy 234.95 113.03))
+    (stroke (width 0) (type default) (color 0 0 0 0))
+  )
   (wire (pts (xy 166.37 113.03) (xy 175.26 113.03))
     (stroke (width 0) (type default) (color 0 0 0 0))
   )
   (wire (pts (xy 157.48 121.92) (xy 157.48 125.73))
+    (stroke (width 0) (type default) (color 0 0 0 0))
+  )
+  (wire (pts (xy 234.95 113.03) (xy 223.52 113.03))
     (stroke (width 0) (type default) (color 0 0 0 0))
   )
@@
     (in_bom yes) (on_board yes) (fields_autoplaced)
     (property "Reference" "J3" (id 0) (at 67.31 48.26 0))
-    (property "Value" "105017-0001" (id 1) (at 67.31 50.8 0))
+    (property "Value" "105017-0001 Micro USB Conn" (id 1) (at 67.31 50.8 0))
     (property "Footprint" "MOLEX_105017-0001" (id 2) (at 67.31 58.42 0)
       (effects (font (size 1.27 1.27)) (justify bottom) hide)
@@
     (in_bom yes) (on_board yes) (fields_autoplaced)
     (property "Reference" "U7" (id 0) (at 207.01 102.87 0))
-    (property "Value" "NCP161ASN330T1G" (id 1) (at 207.01 105.41 0))
+    (property "Value" "NCP161ASN330T1G LDO" (id 1) (at 207.01 105.41 0))
     (property "Footprint" "Components:SOT95P280X145-5N" (id 2) (at 207.01 107.95 0))
     (property "Datasheet" "https://www.mouser.co.uk/datasheet/2/308/1/NCP161_D-2316989.pdf" (id 3) (at 207.01 118.11 0)
@@
     (in_bom yes) (on_board yes) (fields_autoplaced)
     (property "Reference" "J2" (id 0) (at 86.36 106.68 0))
-    (property "Value" "Conn_01x02" (id 1) (at 86.36 109.22 0))
+    (property "Value" "JST_PH_S2B-PH-K_1x02_P2.00mm_Horizontal" (id 1) (at 86.36 109.22 0))
     (property "Footprint" "Components:JST_PH_S2B-PH-K_1x02_P2.00mm_Horizontal" (id 2) (at 86.36 115.57 0)
       (effects (font (size 1.27 1.27)) hide)
@@
     (pin "2")
   )
-  (symbol (lib_id "Device:C_Polarized_Small") (at 234.95 115.57 0) (unit 1)
-    (in_bom yes) (on_board yes) (fields_autoplaced)
-    (property "Reference" "C16" (id 0) (at 237.49 113.7538 0)
-      (effects (font (size 1.27 1.27)) (justify left))
-    )
-    (property "Value" "4.7uF" (id 1) (at 237.49 116.2938 0)
-      (effects (font (size 1.27 1.27)) (justify left))
-    )
-    (property "Footprint" "Capacitor_SMD:C_1206_3216Metric_Pad1.33x1.80mm_HandSolder" (id 2) (at 234.95 115.57 0)
-      (effects (font (size 1.27 1.27)) hide)
-    )
-    (property "Datasheet" "~" (id 3) (at 234.95 115.57 0)
+  (symbol (lib_id "Device:C_Polarized_Small") (at 234.95 116.84 0) (unit 1)
+    (in_bom yes) (on_board yes) (fields_autoplaced)
+    (property "Reference" "C16" (id 0) (at 237.49 115.0238 0)
+      (effects (font (size 1.27 1.27)) (justify left))
+    )
+    (property "Value" "4.7uF Tantalum Capacitor" (id 1) (at 237.49 117.5638 0)
+      (effects (font (size 1.27 1.27)) (justify left))
+    )
+    (property "Footprint" "Capacitor_SMD:C_1206_3216Metric_Pad1.33x1.80mm_HandSolder" (id 2) (at 234.95 116.84 0)
+      (effects (font (size 1.27 1.27)) hide)
+    )
+    (property "Datasheet" "~" (id 3) (at 234.95 116.84 0)
       (effects (font (size 1.27 1.27)) hide)
     )
@@
     (in_bom yes) (on_board yes) (fields_autoplaced)
     (property "Reference" "U5" (id 0) (at 105.9157 40.64 0))
-    (property "Value" "STF202-22T1G" (id 1) (at 105.9157 43.18 0))
+    (property "Value" "STF202-22T1G ESD/EMI Chip" (id 1) (at 105.9157 43.18 0))
     (property "Footprint" "Components:STF202-22T1G" (id 2) (at 105.9157 45.72 0))
     (property "Datasheet" "" (id 3) (at 102.87 66.04 0)
@@
     (in_bom yes) (on_board yes) (fields_autoplaced)
     (property "Reference" "U6" (id 0) (at 156.845 102.87 0))
-    (property "Value" "MAX40203_SOT23" (id 1) (at 156.845 105.41 0))
+    (property "Value" "MAX40203_SOT23 Ideal Diode" (id 1) (at 156.845 105.41 0))
     (property "Footprint" "Package_TO_SOT_SMD:SOT-23-5" (id 2) (at 156.845 107.95 0))
     (property "Datasheet" "" (id 3) (at 156.21 114.3 0)
@@
     (in_bom yes) (on_board yes) (fields_autoplaced)
     (property "Reference" "D1" (id 0) (at 173.0375 54.61 0))
-    (property "Value" "DFLS130L" (id 1) (at 173.0375 57.15 0))
+    (property "Value" "DFLS130L Schottkey Diode" (id 1) (at 173.0375 57.15 0))
     (property "Footprint" "Components:PowerDI123" (id 2) (at 172.72 60.96 0)
       (effects (font (size 1.27 1.27)) hide)
